Commit message: collision works by adding an overlapping link; cage-escape demo

File: models/donut/donut.urdf (robot description, URDF)
Before this commit: robot donut, 1 links, 0 joints
Links:
- added link arm_link1; collision mesh filename=package://donut/donut_col.stl; visual mesh filename=package://donut/donut_vis.dae
Joints:
- added joint joint1: type continuous, parent base_link, child arm_link1, origin xyz=0 0 0 rpy=0 0 0
